Commit message: removed payload

File: urdf/anymal.urdf (robot description, URDF)
Before this commit: robot anymal, 96 links, 95 joints
Links:
- removed link inspection_payload_camera
- removed link inspection_payload_camera_default
- removed link inspection_payload_head
- removed link inspection_payload_light
- removed link inspection_payload_microphone
- removed link inspection_payload_mount
- removed link inspection_payload_pan
- removed link inspection_payload_thermal_camera
- removed link inspection_payload_tilt
Joints:
- removed joint base_to_inspection_payload_mount
- removed joint inspection_payload_head_to_camera
- removed joint inspection_payload_head_to_light
- removed joint inspection_payload_head_to_microphone
- removed joint inspection_payload_head_to_thermal_camera
- removed joint inspection_payload_mount_to_camera_default
- removed joint inspection_payload_mount_to_pan
- removed joint inspection_payload_pan_to_tilt
- removed joint inspection_payload_tilt_to_head

Commit message: Minor fixes

File: urdf/anymal.urdf (robot description, URDF)
Before this commit: robot anymal, 87 links, 86 joints
Links:
- removed link lidar
- added link velodyne_lidar, mass 0.9017; collision cylinder length=0.1355 radius=0.07; visual mesh filename=package://anymal_d_simple_description/meshes/lidar.dae
Joints:
- removed joint lidar_parent_to_lidar
- added joint lidar_parent_to_velodyne_lidar: type fixed, parent lidar_parent, child velodyne_lidar, origin xyz=0 0 0 rpy=0 0 1.5707963267948966

Commit message: Add fixed joint and link for PTSD integration in URDF

File: urdf/anymal.urdf (robot description, URDF)
Before this commit: robot anymal, 87 links, 86 joints
Links:
- added link ptsd_link
Joints:
- added joint base_to_ptsd_link: type fixed, parent base, child ptsd_link, origin xyz=0.1825 0 0.125 rpy=0 0 0
