Commit message: Rename the payload mount frame from ptsd_link to owl_mount
The pan-tilt sensing deck that bolts to this frame is now developed as owl
(owl_description), so the frame carried the superseded project name. owl_mount
also says what it is — a mount point — rather than naming whichever payload
occupies it, matching inspection_payload_mount in the payload variant.

Frame only: an empty link plus its fixed joint on base, no geometry, and no
other file in the repo referenced it. The 0.1825 0 0.125 offset is unchanged,
so the kinematics are identical.

Not owl_link: owl_description already uses that name for the deck's own first
frame, so reusing it here would give one frame two parents.

File: urdf/anymal.urdf (robot description, URDF)
Before this commit: robot anymal, 88 links, 87 joints
Links:
- removed link ptsd_link
- added link owl_mount
Joints:
- removed joint base_to_ptsd_link
- added joint base_to_owl_mount: type fixed, parent base, child owl_mount, origin xyz=0.1825 0 0.125 rpy=0 0 0
